File: Senior Design Debug PCB V1.s#1.sch (EAGLE design)
At the start: 38 parts, among them P00_R 1K, P01_R 1K, P02_R 1K, U1 BLE113-A-VISUAL, U2 TLV70033_DCK_5, U3 TLV70033_DCK_5

Commit message: general layout for PCB, no traces yet
Parts:
- removed BLE_C1, BLE_C2, IMU_C4, USB_C: 4.7 uF, eagle-ltspice:C
- removed CL_C2: 0.1 uF, eagle-ltspice:C
- removed ISET_R, TMR_R: (no value), eagle-ltspice:R
- removed TS_R: 10K, eagle-ltspice:R
- removed USB_INPUT: USB_MICROB_PLUGCONN-11752, SparkFun-Connectors:USB_MICROB_PLUGCONN-11752
- added BLE_PWR_C1, BLE_PWR_C2, BQ_IN_C: 4.7 uF, eagle-ltspice:C
- added BLE_PWR_EN, BQ_CE_JMP, BQ_EN1, BQ_EN2, CL_BYPASS, IMU_PWR_EN, TD_JMP: (no value), jumper:J2X2MM
- added BLE_PWR_JMP, BQ_OUT_JMP, IMU_PWR_JMP: (no value), jumper:JP1E
- added BLE_R1, BQ_ISET_H_R1, BQ_ISET_H_R2, BQ_ISET_H_R3, OUT_R2, TMR_H_R1, TMR_H_R2, TMR_H_R3: (no value), eagle-ltspice:R
- added BLE_R1_JMP, BQ_ISET_JMP, CC_DEBUGGER_JMP, CL_EN, IMU_R1_JMP, OUT_R2_JMP, PGOOD_JMP: 22-23-2021, con-molex:22-23-2021
- added BLE_RST_R: 10K, 50V, 0.063W, eagle-ltspice:R
- added BLE_RST_SW: (no value), SparkFun-Electromechanical:SWITCH-SPDTPTH
- added BQ_ISET_H, TMR_H: (no value), jumper:JP4Q
- added BQ_TS_R: 10K, eagle-ltspice:R
- added CL_C1: 10 uF, eagle-ltspice:C
- added DC_C1: 1.0 µF, eagle-ltspice:C
- added DC_C2: 0.1 µF, eagle-ltspice:C
- added IMU2BLE: (no value), con-lstb:MA05-2
- added IMU_R1: 30 Ω, eagle-ltspice:R
- added JP1: USB_MICROB_PLUG-PTH2, SparkFun-Connectors:USB_MICROB_PLUG-PTH2
- added P22_PAD, TP5: TPB1,27, testpad:TPB1,27
- IMU_C1: value 0.1 µF -> 10 nF
- IMU_C3: value 10 nF -> 4.7 uF
Connections:
- removed net BLE_PWR: BLE_C1.1, BLE_C2.1, CC_PROGRAMMER.2, CC_PROGRAMMER.9, SCL_PU.2, SDA_PU.2, U1.AVDD, U1.DVDD, U3.OUT
- removed net IMU_PWR: IMU_C2.1, IMU_C4.2, MPU-9150.VDD, MPU-9150.VDD13, MPU-9150.VLOGIC, SCL_R.2, SDA_R.2, U2.OUT
- removed net P2_1: CC_PROGRAMMER.4, U1.P2_1
- removed net P2_2: CC_PROGRAMMER.3, U1.P2_2
- removed net SCL: MPU-9150.SCL, SCL_PU.1, SCL_R.1, U1.SCL
- removed net SDA: MPU-9150.SDA, SDA_PU.1, SDA_R.1, U1.SDA
- new net BLE_POWER: BLE_PWR_C1.1, BLE_PWR_C2.1, BLE_PWR_JMP.1, BLE_PWR_JMP.2, BLE_R1.1, BLE_R1_JMP-1.S, SCL_R.2, SDA_R.2, TP5.TP, U3.OUT
- new net IMU_POWER: IMU_PWR_JMP.2, U2.OUT
- new net N$12: CC_DEBUGGER_JMP-1.S, CC_PROGRAMMER.4, U1.P2_1
- new net N$16: IMU_C3.1, IMU_R1.1, IMU_R1_JMP-2.S, MPU-9150.VDD, MPU-9150.VLOGIC
- new net N$18: BLE_RST_R.1, BLE_RST_SW.O
- new net N$20: BQ24230.*CE, BQ_CE_JMP.2
- new net N$21: BQ24230.EN2, BQ_EN2.2
- new net N$27: BQ_OUT_JMP.1, OUT_R2.2, OUT_R2_JMP-2.S
- new net N$30: TMR_H.8, TMR_H_R3.1
- new net N$32: TMR_H.6, TMR_H_R2.1
- new net N$33: TMR_H.4, TMR_H_R1.1
- new net N$34: BLE_PWR_EN.2, U3.EN
- new net N$35: BLE_R1.2, BLE_R1_JMP-2.S, U1.AVDD, U1.DVDD
- new net N$36: IMU_PWR_EN.2, U2.EN
- new net N$37: BQ24230.TD, TD_JMP.2
- new net N$39: BQ_ISET_H.8, BQ_ISET_H_R3.1
- new net N$40: BQ_ISET_H.6, BQ_ISET_H_R2.1
- new net N$41: BQ_ISET_H.4, BQ_ISET_H_R1.1
- new net N$42: BQ_OUT_JMP.2, SBC_OUT_SW.S
- new net N$43: CL_BYPASS.1, CL_C1.1, CL_R1.1, CURR_LIM.VIN
- new net N$47: CL_BYPASS.3, CURR_LIM.VOUT, U2.IN, U3.IN
- new net N$6: BQ24230.EN1, BQ_EN1.2
- new net SCL_9150: IMU2BLE.4, IMU2BLE.8, MPU-9150.SCL, SCL_R.1
- new net SCL_BLE113: IMU2BLE.3, IMU2BLE.7, SCL_PU.2, U1.SCL
- new net SDA_9150: IMU2BLE.10, IMU2BLE.6, MPU-9150.SDA, SDA_R.1
- new net SDA_BLE113: IMU2BLE.5, IMU2BLE.9, SDA_PU.2, U1.SDA
- new net VCC: BQ24230.OUT, BQ24230.OUT_2, CC_PROGRAMMER.9, OUT_C1.2, OUT_R2.1, OUT_R2_JMP-1.S
- net DC_IN: now also BQ_IN_C.2, JP1.VCC; no longer USB_C.1, USB_INPUT.VCC
- net GND: now also BLE_PWR_C1.2, BLE_PWR_C2.2, BLE_PWR_EN.3, BLE_RST_SW.S, BQ_CE_JMP.3, BQ_EN1.3, BQ_EN2.3, BQ_IN_C.1, BQ_ISET_H.2, BQ_ISET_H_R1.2, BQ_ISET_H_R2.2, BQ_ISET_H_R3.2, BQ_ISET_JMP-2.S, BQ_TS_R.1, CC_DEBUGGER_JMP-2.S, CL_C1.2, CL_EN-1.S, DC_C1.2, DC_C2.2, IMU2BLE.1, IMU2BLE.2, IMU_C1.1, IMU_C3.2, IMU_PWR_EN.3, JP1.GND, PGOOD_JMP-2.S, TD_JMP.3, TMR_H.2, TMR_H_R1.2, TMR_H_R2.2, TMR_H_R3.2; no longer BLE_C1.2, BLE_C2.2, BQ24230.*CE, BQ24230.EN1, BQ24230.EN2, BQ24230.TD, CL_C2.2, IMU_C1.2, IMU_C3.1, ISET_R.1, MPU-9150.GND18, TMR_R.2, TS_R.1, USB_C.2, USB_INPUT.GND
- net N$1: now also IMU_C1.2; no longer IMU_C3.2
- net N$15: now also CL_EN-2.S
- net N$17: now also BQ_TS_R.2; no longer TS_R.2
- net N$2: now also BQ_ISET_H.1, BQ_ISET_H.3, BQ_ISET_H.5, BQ_ISET_H.7, BQ_ISET_JMP-1.S; no longer ISET_R.2
- net N$22: now also PGOOD_JMP-1.S
- net N$29: now also CL_BYPASS.2; no longer CL_R1.1, CURR_LIM.VIN
- net N$3: now also IMU_C2.1; no longer IMU_C1.1
- net N$31: now also TMR_H.1, TMR_H.3, TMR_H.5, TMR_H.7; no longer TMR_R.1
- net N$5: now also IMU_PWR_JMP.1, IMU_R1.2, IMU_R1_JMP-1.S; no longer IMU_C4.1
- net N$8: now also CC_PROGRAMMER.3, P22_PAD.TP, U1.P2_2; no longer CL_C2.1, CURR_LIM.VOUT, U2.IN, U3.IN
- net RESET: now also BLE_RST_SW.P, U1.RESET
- net VDD: now also BLE_PWR_EN.1, BLE_RST_R.2, BQ_CE_JMP.1, BQ_EN1.1, BQ_EN2.1, CC_PROGRAMMER.2, DC_C1.1, DC_C2.1, IMU_PWR_EN.1, SCL_PU.1, SDA_PU.1, TD_JMP.1; no longer BQ24230.OUT, BQ24230.OUT_2, OUT_C1.2, SBC_OUT_SW.S, U1.RESET, U2.EN, U3.EN
Other:
- note added: "Physically close to MPU9150"
- note added: "SCL_BLE113"
- note added: "SDA_BLE113"
- note added: "Where is reset going to?"
- moved on the sheet: BATT_C, BATT_CONN, CC_PROGRAMMER, CHG_LED, CHG_R, CL_R1, CURR_LIM, IMU_C1, IMU_C2, IMU_C3, MPU-9150, OUT_C1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
